File: Rev2/GoGoGoRev2.sch (KiCad schematic (older format))
At the start: 0 parts

Commit message: Added TB6593 to schematic
Parts:
- added C? (x4): C, symbol C
- added P? (x2): CONN_01X02, symbol CONN_01X02
- added P?: CONN_01X04, symbol CONN_01X04
- added U?: TB6593FNG, symbol TB6593FNG
Connections:
- new net: P?.2 (P2), U?.14 (O2), U?.15 (O2)
- new net: C?.1, C?.1, U?.16 (VM3), U?.17 (VM4), U?.4 (VM1), U?.5 (VM2)
- new net: P?.3 (P3), U?.18 (IN1)
- new net: P?.2 (P2), U?.19 (IN2)
- new net: P?.1 (P1), U?.2 (PWM)
- new net: C?.1, C?.1, P?.2 (P2), U?.20 (VCC)
- new net: P?.4 (P4), U?.3 (STBY)
- new net: P?.1 (P1), U?.6 (O1), U?.7 (O1)
- new net GND: C?.2, C?.2, C?.2, C?.2, P?.1 (P1), U?.1 (GND), U?.10 (PGND3), U?.11 (PGND4), U?.12 (PGND5), U?.13 (PGND6), U?.8 (PGND1), U?.9 (PGND2)
