File: Rev2/GoGoGoRev2.sch (KiCad schematic (older format))
At the start: 8 parts, among them P1 CONN_01X02, P2 CONN_01X04, P3 CONN_01X02, U1 TB6593FNG

Commit message: Finished layout
Connections:
- net O2: now reaches P3.2 (P2), U1.14 (O2), U1.15 (O2)
- net VM: now reaches C3.1, C4.1, U1.16 (VM3), U1.17 (VM4), U1.4 (VM1), U1.5 (VM2)
- net IN1: now reaches P2.3 (P3), U1.18 (IN1)
- net IN2: now reaches P2.2 (P2), U1.19 (IN2)
- net PWM: now reaches P2.1 (P1), U1.2 (PWM)
- net VCC: now reaches C1.1, C2.1, P1.2 (P2), U1.20 (VCC)
- net STBY: now reaches P2.4 (P4), U1.3 (STBY)
- net O1: now reaches P3.1 (P1), U1.6 (O1), U1.7 (O1)
Changed lines of the file:
@@
 Wire Wire Line
 	4750 2900 3950 2900
+Text Label 4600 1900 0    60   ~ 0
+VCC
+Text Label 7100 2000 0    60   ~ 0
+VM
+Text Label 6950 3050 0    60   ~ 0
+O1
+Text Label 6950 3250 0    60   ~ 0
+O2
+Text Label 4400 2800 0    60   ~ 0
+STBY
+Text Label 4400 2900 0    60   ~ 0
+IN1
+Text Label 4400 3000 0    60   ~ 0
+IN2
+Text Label 4500 3450 0    60   ~ 0
+PWM
+Text Label 6850 3750 0    60   ~ 0
+PGND
 $EndSCHEMATC

Commit message: updated part numbers
Parts:
- U1: Link (none) -> http://parts.io/detail/1775277/TB6593FNG; MPN (none) -> TB6593FNG
Changed lines of the file:
@@
 F 2 "SMD_Packages:SSOP-20" H 4800 3850 60  0001 C CNN
 F 3 "" H 4800 3850 60  0000 C CNN
+F 4 "TB6593FNG" H 5850 3250 60  0001 C CNN "MPN"
+F 5 "http://parts.io/detail/1775277/TB6593FNG" H 5850 3250 60  0001 C CNN "Link"
 	1    5850 3250
 	1    0    0    -1
