File: MotorEncoderBoard/MotorEncoderBoard.kicad_pcb (KiCad board)
At the start: 2 copper layers, 11 parts, among them P1 CONN_01X02, P2 CONN_01X02, U1 RPI-579N1, U2 LM311N

Commit message: Finished PCB and generated Gerbers
Parts:
- TP1: footprint Measurement_Points:Measurement_Point_Round-SMD-Pad_Big -> Measurement_Points:Measurement_Point_Round-SMD-Pad_Small
- moved TP1 0.76 mm to (172.5, 88.9)
Routing:
- net Net-(R2-Pad2): track 18.2 -> 21.4 mm
Other:
- board outline added: 26.2 x 19 mm
Changed lines of the file:
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@@
   (general
     (links 22)
-    (no_connects 12)
-    (area 0 0 0 0)
+    (no_connects 0)
+    (area 149.323734 82.506 176.072001 102.666001)
     (thickness 1.6)
-    (drawings 0)
-    (tracks 42)
+    (drawings 4)
+    (tracks 44)
     (zones 0)
     (modules 11)
@@
     (visible_elements FFFEFF7F)
     (pcbplotparams
-      (layerselection 0x00030_80000001)
+      (layerselection 0x010fc_80000001)
       (usegerberextensions false)
       (excludeedgelayer true)
@@
       (psa4output false)
       (plotreference true)
-      (plotvalue true)
+      (plotvalue false)
       (plotinvisibletext false)
       (padsonsilk false)
-      (subtractmaskfromsilk false)
+      (subtractmaskfromsilk true)
       (outputformat 1)
       (mirror false)
-      (drillshape 1)
+      (drillshape 0)
       (scaleselection 1)
-      (outputdirectory ""))
+      (outputdirectory Gerbers/))
   )
   (net 0 "")
@@
     )
   )
-  (module Measurement_Points:Measurement_Point_Round-SMD-Pad_Big (layer F.Cu)
-    (at 173.228 88.9508)
-    (descr "Mesurement Point, Round, SMD Pad, DM 3mm,")
-    (tags "Mesurement Point, Round, SMD Pad, DM 3mm,")
-    (fp_text reference TP1 (at 1.27 1.9812) (layer F.SilkS)
-      (effects (font (size 0.5 0.5) (thickness 0.1)))
-    )
-    (fp_text value OptoOut (at 2.54 3.81) (layer F.Fab)
-      (effects (font (size 0.5 0.5) (thickness 0.1)))
-    )
-    (pad 1 smd circle (at 0 0) (size 2.99974 2.99974) (layers F.Cu F.Paste F.Mask)
-      (net 5 "Net-(R2-Pad2)"))
-  )
   (module Housings_SOIC:SOIC-8_3.9x4.9mm_Pitch1.27mm (layer F.Cu)
     (at 160.6804 94.9452)
@@
       (net 2 GND))
   )
-  (segment (start 152.8788 93.5736) (end 152.8788 92.122) (width 0.6096) (layer F.Cu) (net 1) (status 400000))
+  (module Measurement_Points:Measurement_Point_Round-SMD-Pad_Small (layer F.Cu)
+    (at 172.466 88.9)
+    (descr "Mesurement Point, Round, SMD Pad, DM 1.5mm,")
+    (tags "Mesurement Point, Round, SMD Pad, DM 1.5mm,")
+    (fp_text reference TP1 (at -0.254 -1.524) (layer F.SilkS)
+      (effects (font (size 0.5 0.5) (thickness 0.1)))
+    )
+    (fp_text value OptoOut (at 1.27 2.54) (layer F.Fab)
+      (effects (font (size 0.5 0.5) (thickness 0.1)))
+    )
+    (pad 1 smd circle (at 0 0) (size 1.524 1.524) (layers F.Cu F.Paste F.Mask)
+      (net 5 "Net-(R2-Pad2)"))
+  )
+  (gr_line (start 176.022 83.566) (end 149.86 83.566) (angle 90) (layer Edge.Cuts) (width 0.1))
+  (gr_line (start 176.022 102.616) (end 176.022 83.566) (angle 90) (layer Edge.Cuts) (width 0.1))
+  (gr_line (start 149.86 102.616) (end 176.022 102.616) (angle 90) (layer Edge.Cuts) (width 0.1))
+  (gr_line (start 149.86 83.566) (end 149.86 102.616) (angle 90) (layer Edge.Cuts) (width 0.1))
+  (segment (start 152.8788 93.5736) (end 152.8788 92.122) (width 0.6096) (layer F.Cu) (net 1))
   (via (at 152.8064 92.0496) (size 0.6858) (layers F.Cu B.Cu) (net 1))
   (segment (start 152.8788 92.122) (end 152.8064 92.0496) (width 0.6096) (layer F.Cu) (net 1))
@@
   (segment (start 157.6324 98.806) (end 158.3436 98.0948) (width 0.6096) (layer F.Cu) (net 3))
   (segment (start 155.8836 88.9) (end 159.2745 88.9) (width 0.6096) (layer F.Cu) (net 4))
+  (segment (start 172.466 88.9) (end 169.2745 88.9) (width 0.6096) (layer F.Cu) (net 5))
+  (segment (start 169.3253 88.9508) (end 169.2745 88.9) (width 0.6096) (layer F.Cu) (net 5))
   (segment (start 170.0568 92.0496) (end 170.0568 89.6823) (width 0.6096) (layer F.Cu) (net 5))
   (segment (start 170.0568 89.6823) (end 169.2745 88.9) (width 0.6096) (layer F.Cu) (net 5))
@@
   (segment (start 160.782 91.694) (end 160.782 93.6752) (width 0.6096) (layer F.Cu) (net 5))
   (segment (start 163.576 88.9) (end 160.782 91.694) (width 0.6096) (layer F.Cu) (net 5))
-  (segment (start 155.5788 93.5736) (end 155.5788 95.5548) (width 0.6096) (layer F.Cu) (net 6) (status C00000))
-  (segment (start 155.5788 95.5548) (end 155.6296 95.6056) (width 0.6096) (layer F.Cu) (net 6) (status C00000))
+  (segment (start 155.5788 93.5736) (end 155.5788 95.5548) (width 0.6096) (layer F.Cu) (net 6))
+  (segment (start 155.5788 95.5548) (end 155.6296 95.6056) (width 0.6096) (layer F.Cu) (net 6))
   (segment (start 155.6296 95.6056) (end 157.955 95.6056) (width 0.6096) (layer F.Cu) (net 6))
   (segment (start 157.955 95.6056) (end 157.9804 95.5802) (width 0.6096) (layer F.Cu) (net 6))
@@
     (connect_pads (clearance 0.1524))
     (min_thickness 0.1524)
-    (fill (arc_segments 16) (thermal_gap 0.254) (thermal_bridge_width 0.254))
+    (fill yes (arc_segments 16) (thermal_gap 0.254) (thermal_bridge_width 0.254))
     (polygon
       (pts
-        (xy 181.8005 102.235) (xy 149.606 102.235) (xy 149.606 76.708) (xy 181.8005 76.708)
+        (xy 176.022 102.616) (xy 149.86 102.616) (xy 149.86 83.566) (xy 176.022 83.566)
       )
     )
@@
     (connect_pads (clearance 0.1524))
     (min_thickness 0.1524)
-    (fill (arc_segments 16) (thermal_gap 0.254) (thermal_bridge_width 0.254))
+    (fill yes (arc_segments 16) (thermal_gap 0.254) (thermal_bridge_width 0.254))
     (polygon
       (pts
-        (xy 149.606 76.708) (xy 149.606 102.235) (xy 181.8005 102.235) (xy 181.8005 76.7715) (xy 149.606 76.708)
+        (xy 176.022 102.616) (xy 149.86 102.616) (xy 149.86 83.566) (xy 176.022 83.566)
       )
     )
