File: Rev1/GoGoGo-Rev1.kicad_pcb (KiCad board)
At the start: 2 copper layers, 14 x 13.2 mm, 6 parts, among them P1 CONN_01X03, P2 CONN_01X02, P3 CONN_01X03, U1 DRV8837DSGR

Commit message: Updated fill zones to get better copper coverage
Parts:
- moved C1 0.25 mm to (136.7, 104.4)
- moved P2 0.25 mm to (142.0, 105.4)
Routing:
- net /VM: track 7.79 -> 0.00 mm
- net /OUT1: track 4.10 -> 0.00 mm
- net /OUT2: track 3.99 -> 0.00 mm
- added copper zone on F.Cu, net /OUT1
- added copper zone on F.Cu, net /OUT2
